File: CAD/stlink-v3-hwmod.brd (EAGLE design)
At the start: 32 x 48 mm, 10 parts, among them U1 STLINK-V3MODS

Commit message: Final revision.
Created Gerbers,
Ready for production
Parts:
- added H1, H2: MOUNT-HOLE3.2, holes:3,2
- added U$1: STLINK-V3-HWMODS, Logo-hwtronics:STLINK-V3-HWMODS
- moved J1 2.86 mm to (16.0, 7.00)
- moved J4 2.50 mm to (3.50, 14.5)
- moved J7 2.50 mm to (28.5, 14.5)
- moved LOGO1 1.50 mm to (25.0, 2.00)
- moved J2 1.00 mm to (22.2, 21.0)
- moved J8 1.00 mm to (28.5, 18.0)
Routing:
- net T_SWCLK: track 32.8 -> 37.1 mm
- net T_GND: track 45.8 -> 49.7 mm
- net T_VCC: track 34.0 -> 37.9 mm
- net T_NRST: track 42.0 -> 45.5 mm
- net GND: track 0.00 -> 3.43 mm, vias 0 -> 41
- net T_SWDIO: track 29.5 -> 32.5 mm
- net VCP_RX: track 21.1 -> 18.6 mm
- net I2C_SCL: track 36.1 -> 38.5 mm
- net T_SWO: track 24.5 -> 26.9 mm
- net VCP_TX: track 22.4 -> 20.1 mm
- net I2C_SDA: track 17.6 -> 15.4 mm
- net GPIO0: track 11.6 -> 10.2 mm
- net GPIO1: track 10.1 -> 8.92 mm
- net +5V: track 53.9 -> 52.8 mm
Other:
- board size 32 x 48 mm -> 32 x 54.5 mm
- board text added: "2020-04"
- board text added: "5V"
- board text added: "CLK"
- board text added: "CTS"
- board text added: "Designed by: @hwtronics"
- board text added: "Docs & Source:"
- board text added: "GND"
- board text added: "GPIO0"
- board text added: "GPIO1"
- board text added: "GPIO2"
- board text added: "GPIO3"
- board text added: "MISO"
- board text added: "MOSI"
- board text added: "NSS"
- board text added: "RTS"
- board text added: "RX"
- board text added: "Rev. A"
- board text added: "SCL"
- board text added: "SDA"
- board text added: "STLINK-V3 HWMODS"
- board text added: "TX"
- board text added: "https://hwtronics.com"
