File: CAD/stlink-v3-hwmod.sch (EAGLE design)
At the start: 10 parts, among them U1 STLINK-V3MODS

Commit message: Final revision.
Created Gerbers,
Ready for production
Parts:
- added H1, H2: MOUNT-HOLE3.2, holes:MOUNT-HOLE3.2
- added U$1: STLINK-V3-HWMODS, Logo-hwtronics:STLINK-V3-HWMODS
Changed lines of the file:
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@@
 <part name="J8" library="SparkFun-Connectors" library_urn="urn:adsk.eagle:library:513" deviceset="CONN_06" device="SILK_FEMALE_PTH" package3d_urn="urn:adsk.eagle:package:38009/1"/>
 <part name="LOGO1" library="Logo-hwtronics" deviceset="LOGO-HWTRONICS" device="-10MM"/>
+<part name="H1" library="holes" library_urn="urn:adsk.eagle:library:237" deviceset="MOUNT-HOLE" device="3.2" package3d_urn="urn:adsk.eagle:package:14275/1"/>
+<part name="H2" library="holes" library_urn="urn:adsk.eagle:library:237" deviceset="MOUNT-HOLE" device="3.2" package3d_urn="urn:adsk.eagle:package:14275/1"/>
+<part name="U$1" library="Logo-hwtronics" deviceset="STLINK-V3-HWMODS" device=""/>
 </parts>
 <sheets>
@@
 </instance>
 <instance part="LOGO1" gate="G$1" x="21.59" y="11.43" smashed="yes"/>
+<instance part="H1" gate="G$1" x="124.46" y="17.78" smashed="yes">
+<attribute name="NAME" x="126.492" y="18.3642" size="1.778" layer="95"/>
+<attribute name="VALUE" x="126.492" y="15.3162" size="1.778" layer="96"/>
+</instance>
+<instance part="H2" gate="G$1" x="124.46" y="10.16" smashed="yes">
+<attribute name="NAME" x="126.492" y="10.7442" size="1.778" layer="95"/>
+<attribute name="VALUE" x="126.492" y="7.6962" size="1.778" layer="96"/>
+</instance>
+<instance part="U$1" gate="G$1" x="20.32" y="7.62" smashed="yes"/>
 </instances>
 <busses>
